File: 29F160 to UV EPROM/29F160_to_27C322_2-0.kicad_pcb (KiCad board)
At the start: 4 copper layers, 54.4 x 17.8 mm, 14 parts, among them U1 27C322, U2 29F160, U3 29F160, U4 74LS139

Commit message: Add files via upload
Parts:
- added TP3: TPB1,27, TestPoint:TestPoint_Pad_1.0x1.0mm, F.Cu at (183.8, 102.0)
Routing:
- net GND: track 74.0 -> 64.2 mm
Other:
- board text added: "~{BYTE}"

Commit message: Add files via upload
Parts:
- added TP4: TPB1,27, Bucketmouse:TestPoint_THTPad_D1.5mm_Drill0.7mm, F.Cu at (223.5, 94.0)
- moved C1 1.10 mm to (223.5, 97.2), turned to 0 degrees
- renumbered U1 to P1
Routing:
- net +5V: track 97.5 -> 94.6 mm
- net /~{BYTE}: track 77.1 -> 79.9 mm
- net /D11: track 69.8 -> 70.5 mm
- net GND: track 64.2 -> 63.7 mm, vias 23 -> 21
Other:
- board text added: "P32"

Commit message: Add files via upload
Parts:
- removed JP2: Jumper_3_Open, Jumper:SolderJumper-3_P1.3mm_Open_Pad1.0x1.5mm
- removed TP3: TPB1,27, TestPoint:TestPoint_Pad_1.0x1.0mm
- added RA2: 100k, Bucketmouse:R_0603_1608Metric_Boxed, F.Cu at (185.6, 101.2)
- added RB2: 100k, Bucketmouse:R_0603_1608Metric_Boxed, F.Cu at (185.6, 102.7)
- added RC2: 0, Bucketmouse:R_0603_1608Metric_Boxed, F.Cu at (184.8, 102.0)
- moved G*** 0.08 mm to (191.0, 102.0)
- renumbered R2 to R3
Routing:
- net +5V: track 94.6 -> 92.2 mm
Other:
- board text added: "R2"
