File: 29F160 to UV EPROM/29F160_to_27C322_2-0.kicad_sch (KiCad schematic)
At the start: 12 parts, among them U1 27C322, U2 29F160, U3 29F160, U4 74LS139

Commit message: Add files via upload
Parts:
- added TP3: TPB1,27, TestPoint:TestPoint_Pad_1.0x1.0mm, symbol Connector:TestPoint
Connections:
- net A20: now also TP3.1
Other:
- moved on the sheet: JP2

Commit message: Add files via upload
Parts:
- added TP4: TPB1,27, Bucketmouse:TestPoint_THTPad_D1.5mm_Drill0.7mm, symbol Connector:TestPoint
- renumbered U1 to P1
Connections:
- net ~{BYTE}: now also TP4.1
Other:
- moved on the sheet: R1, R2, TP1, TP2

Commit message: Add files via upload
Parts:
- removed JP2: Jumper_3_Open, Jumper:SolderJumper-3_P1.3mm_Open_Pad1.0x1.5mm, symbol Jumper:Jumper_3_Open
- removed TP3: TPB1,27, TestPoint:TestPoint_Pad_1.0x1.0mm, symbol Connector:TestPoint
- added RA2, RB2: 100k, Bucketmouse:R_0603_1608Metric_Boxed, symbol Device:R
- added RC2: 0, Bucketmouse:R_0603_1608Metric_Boxed, symbol Device:R
- renumbered R2 to R3
Connections:
- net +5V: now also RB2.1
- net A20: now also RC2.1
- net GND: now also RA2.2
- net ~{BYTE}: now also RA2.1, RB2.2, RC2.2
